Commit message: changes

File: dexterous/urdf/hand.urdf (robot description, URDF)
Before this commit: robot HandAssembly, 10 links, 9 joints
Links:
- link base_link: mass 279.34 -> 279.343309739745; geometry collision mesh filename=package://dexterous/meshes/base_link.STL; visual mesh filename=package://dexterous/meshes/base_link.STL
- link finger_1: mass 2.6229 -> 2.6229121926556; geometry collision mesh filename=package://dexterous/meshes/finger_1.STL; visual mesh filename=package://dexterous/meshes/finger_1.STL
- link finger_1_1: mass 2.3997 -> 2.39970738830488; geometry collision mesh filename=package://dexterous/meshes/finger_1_1.STL; visual mesh filename=package://dexterous/meshes/finger_1_1.STL
- link finger_1_1_1: mass 0.67086 -> 0.67086342261683; geometry collision mesh filename=package://dexterous/meshes/finger_1_1_1.STL; visual mesh filename=package://dexterous/meshes/finger_1_1_1.STL
- link finger_2: mass 2.6229 -> 2.62291216260929; geometry collision mesh filename=package://dexterous/meshes/finger_2.STL; visual mesh filename=package://dexterous/meshes/finger_2.STL
- link finger_2_1: mass 2.3997 -> 2.39969803744161; geometry collision mesh filename=package://dexterous/meshes/finger_2_1.STL; visual mesh filename=package://dexterous/meshes/finger_2_1.STL
- link finger_2_1_1: mass 0.67086 -> 0.670866844724945; geometry collision mesh filename=package://dexterous/meshes/finger_2_1_1.STL; visual mesh filename=package://dexterous/meshes/finger_2_1_1.STL
- link finger_3: mass 2.6229 -> 2.62291219958027; geometry collision mesh filename=package://dexterous/meshes/finger_3.STL; visual mesh filename=package://dexterous/meshes/finger_3.STL
- link finger_3_1: mass 2.3997 -> 2.3996917545326; geometry collision mesh filename=package://dexterous/meshes/finger_3_1.STL; visual mesh filename=package://dexterous/meshes/finger_3_1.STL
- link finger_3_1_1: mass 0.67086 -> 0.670863404845149; geometry collision mesh filename=package://dexterous/meshes/finger_3_1_1.STL; visual mesh filename=package://dexterous/meshes/finger_3_1_1.STL
Joints:
- joint fin1: limit lower=0 upper=2 effort=0 velocity=0 -> lower=-1 upper=1 effort=0 velocity=0; origin xyz=0.30864 -0.175 -1.2226 rpy=0 0.58249 0 -> xyz=0.30864 0.175 1.2226 rpy=3.1416 -0.58249 0
- joint fin1_1: limit lower=0 upper=2 effort=0 velocity=0 -> lower=0 upper=1.2 effort=0 velocity=0; origin xyz=0.18245 0.019102 0.034754 rpy=-1.5708 -0.57999 0.10432 -> xyz=0.179538449644514 -1.07387640339573E-05 0.0396629523318704 rpy=-1.5707963267949 -0.582486578802211 -5.9813179065596E-05
- joint fin1_1_1: limit lower=0 upper=2 effort=0 velocity=0 -> lower=-1.5708 upper=0 effort=0 velocity=0; origin xyz=0.17907 -0.1614 0 rpy=0 0 0 -> xyz=0.212076291309529 0.122256317843988 0 rpy=0 0 0
- joint fin2: limit lower=0 upper=2 effort=0 velocity=0 -> lower=-1 upper=1 effort=0 velocity=0; origin xyz=0.38255 0 -0.78051 rpy=0 -0.43641 0 -> xyz=0.38255 0 0.78051 rpy=3.1416 0.43641 0
- joint fin2_1: limit lower=0 upper=2 effort=0 velocity=0 -> lower=-1.2 upper=0 effort=0 velocity=0; origin xyz=0.18145 0.0055277 0.044234 rpy=-1.5708 0.43624 0.030455 -> xyz=0.179526432571969 0.000764504714627967 0.0400025631184961 rpy=-1.5707963267949 0.436410170153714 0.00425842636341441
- joint fin2_1_1: limit lower=0 upper=2 effort=0 velocity=0 -> lower=0 upper=1.5708 effort=0 velocity=0; origin xyz=0.21061 0.11129 0 rpy=0 0 0 -> xyz=0.221690121359748 -0.103809243324189 0 rpy=0 0 0
- joint fin3: limit lower=0 upper=2 effort=0 velocity=0 -> lower=-1 upper=1 effort=0 velocity=0; origin xyz=0.30864 0.175 -1.2226 rpy=0 0.58249 0 -> xyz=0.308639953146715 -0.175000000000232 1.2225627998667 rpy=3.14159265358979 -0.58248657962397 0
- joint fin3_1: limit lower=0 upper=2 effort=0 velocity=0 -> lower=0 upper=1.2 effort=0 velocity=0; origin xyz=0.18357 0.000728 0.034717 rpy=-1.5708 -0.58248 0.0039657 -> xyz=0.179528666620996 -0.00199234467872766 0.0396429453369453 rpy=-1.5707963267949 -0.582458293086268 -0.0110971853921247
- joint fin3_1_1: limit lower=0 upper=2 effort=0 velocity=0 -> lower=0 upper=1.5708 effort=0 velocity=0; origin xyz=0.17633 -0.16546 0 rpy=0 0 0 -> xyz=0.212632639805716 0.121302703469605 0 rpy=0 0 0
