Commit message: Ya jala el control de posicion de los 3 dedos huhuhuhuu

File: Dexterous/dexterous/urdf/hand5.urdf (robot description, URDF)
Before this commit: robot dexterous, 13 links, 12 joints
Joints:
- joint fin2: origin xyz=0.338191099465507 0 0.774632196937085 rpy=3.14159265358979 0.194237175479863 0 -> xyz=0.338191099465507 0 0.774632196937085 rpy=0 0.194237175479863 0
- joint fin2_1: origin xyz=0.179528059776071 0 0 rpy=1.5707963267949 0 0 -> xyz=0.179528059776071 0 0 rpy=-1.5707963267949 0 0
