Commit message: Fixed new URDF with espherical fingertips

File: Dexterous/dexterous/urdf/hand.urdf (robot description, URDF)
Before this commit: robot hand, 10 links, 9 joints
Links:
- added link finger_1_eef, mass 1.2195909202896; collision mesh filename=package://dexterous/meshes/finger_1_eef.STL; visual mesh filename=package://dexterous/meshes/finger_1_eef.STL
- added link finger_2_eef, mass 1.21958916107902; collision mesh filename=package://dexterous/meshes/finger_2_eef.STL; visual mesh filename=package://dexterous/meshes/finger_2_eef.STL
- added link finger_3_eef, mass 1.21959092028959; collision mesh filename=package://dexterous/meshes/finger_3_eef.STL; visual mesh filename=package://dexterous/meshes/finger_3_eef.STL
- link finger_1: mass 2.6229121926556 -> 2.62291219261926
- link finger_1_1: mass 2.39970738830488 -> 2.39969138530032
- link finger_1_1_1: mass 0.67086342261683 -> 1.2195909202896
- link finger_2: mass 2.62291216260929 -> 2.62291216939468
- link finger_2_1: mass 2.39969803744161 -> 2.39968898922773
- link finger_2_1_1: mass 0.670866844724945 -> 1.21958916107902
- link finger_3: mass 2.62291219958027 -> 2.62291219261926
- link finger_3_1: mass 2.3996917545326 -> 2.39969138530032
- link finger_3_1_1: mass 0.670863404845149 -> 1.21959092028959
Joints:
- added joint fin1_eef: type fixed, parent finger_1_1_1, child finger_1_eef, origin xyz=0.0339613042533951 0.0223712682666903 0 rpy=1.5707963267949 0 0, axis 0 0 0
- added joint fin2_eef: type fixed, parent finger_2_1_1, child finger_2_eef, origin xyz=0.0368558547051152 -0.0171898168811461 0 rpy=1.5707963267949 0 0, axis 0 0 0
- added joint fin3_eef: type fixed, parent finger_3_1_1, child finger_3_eef, origin xyz=0.0339613042533951 0.0223712682666903 0 rpy=1.5707963267949 0 0, axis 0 0 0
- joint fin1: origin xyz=0.30864 0.175 1.2226 rpy=3.1416 -0.58249 0 -> xyz=0.308639953146409 0.175 1.22256279986678 rpy=3.14159265358979 -0.582486579623969 0
- joint fin1_1: axis 0 0 -1 -> -4.99498279141106E-05 -3.29033596607708E-05 -0.999999998211192; limit lower=0 upper=1.2 effort=0 velocity=0 -> lower=0 upper=2 effort=0 velocity=0; origin xyz=0.179538449644514 -1.07387640339573E-05 0.0396629523318704 rpy=-1.5707963267949 -0.582486578802211 -5.9813179065596E-05 -> xyz=0.179528059776071 0 0.0399996964134806 rpy=-1.5707963267949 -0.582486579623969 0
- joint fin1_1_1: axis 0 0 1 -> 4.99498279133785E-05 3.29033596622835E-05 0.999999998211192; limit lower=-1.5708 upper=0 effort=0 velocity=0 -> lower=-2 upper=0 effort=0 velocity=0; origin xyz=0.212076291309529 0.122256317843988 0 rpy=0 0 0 -> xyz=0.204435726444991 0.134667212398081 0 rpy=0 0 0
- joint fin2: origin xyz=0.38255 0 0.78051 rpy=3.1416 0.43641 0 -> xyz=0.382548654972508 0 0.780508398722002 rpy=3.14159265358979 0.436413643527903 0
- joint fin2_1: limit lower=-1.2 upper=0 effort=0 velocity=0 -> lower=-2 upper=0 effort=0 velocity=0; origin xyz=0.179526432571969 0.000764504714627967 0.0400025631184961 rpy=-1.5707963267949 0.436410170153714 0.00425842636341441 -> xyz=0.179528059776071 0 0.0399996964134798 rpy=-1.5707963267949 0.436413643527903 0
- joint fin2_1_1: limit lower=0 upper=1.5708 effort=0 velocity=0 -> lower=0 upper=2 effort=0 velocity=0; origin xyz=0.221690121359748 -0.103809243324189 0 rpy=0 0 0 -> xyz=0.221859646346035 -0.103477155282569 0 rpy=0 0 0
- joint fin3: origin xyz=0.308639953146715 -0.175000000000232 1.2225627998667 rpy=3.14159265358979 -0.58248657962397 0 -> xyz=0.308639953146409 -0.175 1.22256279986678 rpy=3.14159265358979 -0.58248657962397 0
- joint fin3_1: limit lower=0 upper=1.2 effort=0 velocity=0 -> lower=0 upper=2 effort=0 velocity=0; origin xyz=0.179528666620996 -0.00199234467872766 0.0396429453369453 rpy=-1.5707963267949 -0.582458293086268 -0.0110971853921247 -> xyz=0.179528059776071 0 0.03999969641348 rpy=-1.5707963267949 -0.58248657962397 0
- joint fin3_1_1: limit lower=0 upper=1.5708 effort=0 velocity=0 -> lower=0 upper=2 effort=0 velocity=0; origin xyz=0.212632639805716 0.121302703469605 0 rpy=0 0 0 -> xyz=0.20443572644499 0.13466721239808 0 rpy=0 0 0

Commit message: Control de posicion con referencia de los puntos del prisma

File: Dexterous/dexterous/urdf/hand.urdf (robot description, URDF)
Before this commit: robot hand, 13 links, 12 joints
Links:
- link base_link: mass 279.343309739745 -> 225.175136389995
- link finger_1: mass 2.62291219261926 -> 2.62291217240702
- link finger_1_1: mass 2.39969138530032 -> 2.39969201778968
- link finger_1_1_1: mass 1.2195909202896 -> 1.9242557493213
- link finger_1_eef: mass 1.2195909202896 -> 1.9242557493213
- link finger_2: mass 2.62291216939468 -> 2.62290642499631
- link finger_2_1: mass 2.39968898922773 -> 2.39970392286082
- link finger_2_1_1: mass 1.21958916107902 -> 1.92424517665912
- link finger_2_eef: mass 1.21958916107902 -> 1.92424517665912
- link finger_3: mass 2.62291219261926 -> 2.62291217240701
- link finger_3_1: mass 2.39969138530032 -> 2.39969201778967
- link finger_3_1_1: mass 1.21959092028959 -> 1.92425574932128
- link finger_3_eef: mass 1.21959092028959 -> 1.92425574932128
Joints:
- joint fin1: origin xyz=0.308639953146409 0.175 1.22256279986678 rpy=3.14159265358979 -0.582486579623969 0 -> xyz=0.292117822710978 0.175 1.14406683612052 rpy=-3.14159265358979 -0.434081521732677 0
- joint fin1_1: axis -4.99498279141106E-05 -3.29033596607708E-05 -0.999999998211192 -> -5.91557224570015E-05 0 -0.999999998211192; limit lower=0 upper=2 effort=0 velocity=0 -> lower=0 upper=1.65 effort=0 velocity=0; origin xyz=0.179528059776071 0 0.0399996964134806 rpy=-1.5707963267949 -0.582486579623969 0 -> xyz=0.179528059776071 0 0 rpy=-1.5707963267949 0 0
- joint fin1_1_1: axis 4.99498279133785E-05 3.29033596622835E-05 0.999999998211192 -> 5.91557224571689E-05 0 0.999999998211192; limit lower=-2 upper=0 effort=0 velocity=0 -> lower=0 upper=2 effort=0 velocity=0; origin xyz=0.204435726444991 0.134667212398081 0 rpy=0 0 0 -> xyz=0.235471940223928 0 0 rpy=3.14159265358979 0 0
- joint fin1_eef: origin xyz=0.0339613042533951 0.0223712682666903 0 rpy=1.5707963267949 0 0 -> xyz=0.205 0 0 rpy=1.5707963267949 0 0
- joint fin2: origin xyz=0.382548654972508 0 0.780508398722002 rpy=3.14159265358979 0.436413643527903 0 -> xyz=0.338191099465507 0 0.774632196937085 rpy=0 0.194237175479863 0
- joint fin2_1: limit lower=-2 upper=0 effort=0 velocity=0 -> lower=0 upper=1.65 effort=0 velocity=0; origin xyz=0.179528059776071 0 0.0399996964134798 rpy=-1.5707963267949 0.436413643527903 0 -> xyz=0.179528059776071 0 0 rpy=-1.5707963267949 0 0
- joint fin2_1_1: origin xyz=0.221859646346035 -0.103477155282569 0 rpy=0 0 0 -> xyz=0.235471940223929 0 0 rpy=3.14159265358979 0 0
- joint fin2_eef: origin xyz=0.0368558547051152 -0.0171898168811461 0 rpy=1.5707963267949 0 0 -> xyz=0.205 0 0 rpy=1.5707963267949 0 0
- joint fin3: origin xyz=0.308639953146409 -0.175 1.22256279986678 rpy=3.14159265358979 -0.58248657962397 0 -> xyz=0.292117822710978 -0.175 1.14406683612052 rpy=3.14159265358979 -0.434081521732677 0
- joint fin3_1: limit lower=0 upper=2 effort=0 velocity=0 -> lower=0 upper=1.65 effort=0 velocity=0; origin xyz=0.179528059776071 0 0.03999969641348 rpy=-1.5707963267949 -0.58248657962397 0 -> xyz=0.179528059776072 0 0 rpy=-1.5707963267949 0 0
- joint fin3_1_1: origin xyz=0.20443572644499 0.13466721239808 0 rpy=0 0 0 -> xyz=0.235471940223929 0 0 rpy=0 0 0
- joint fin3_eef: origin xyz=0.0339613042533951 0.0223712682666903 0 rpy=1.5707963267949 0 0 -> xyz=0.205 0 0 rpy=1.5707963267949 0 0

Commit message: cositas chidas

File: Dexterous/dexterous/urdf/hand.urdf (robot description, URDF)
Before this commit: robot dexterous, 13 links, 12 joints
Links:
- added link e3, mass 1.3922; collision mesh filename=package://dexterous/meshes/e3.STL; visual mesh filename=package://dexterous/meshes/e3.STL
Joints:
- added joint e_3: type fixed, parent base_link, child e3, origin xyz=0 0 0 rpy=0 0 0, axis 0 0 0

Commit message: Working Project!

File: Dexterous/dexterous/urdf/hand.urdf (robot description, URDF)
Before this commit: robot hand, 14 links, 13 joints
Links:
- link e3: geometry collision mesh filename=package://dexterous/meshes/e3.STL
- link finger_1_eef: geometry 
- link finger_2_eef: geometry 
- link finger_3_eef: geometry 

File: Dexterous/dexterous/urdf/pencil.urdf (robot description, URDF)
Before this commit: robot pencil, 3 links, 2 joints
Links:
- removed link /pencil_robot/base_link
- removed link /pencil_robot/point_link
- added link base_link, mass 0.014148; collision mesh filename=package://dexterous/meshes/base_link_pencil.STL scale=10 10 10; visual mesh filename=package://dexterous/meshes/Pencil.dae
- added link point_link, mass 4.7313E-05; collision mesh filename=package://dexterous/meshes/point_link.STL; visual mesh filename=package://dexterous/meshes/point_link.STL
Joints:
- joint /point_joint: child /pencil_robot/point_link -> point_link; parent /pencil_robot/base_link -> base_link
- joint base_footprint_joint: child /pencil_robot/base_link -> base_link
